Commit message: definitivo

File: snake_description2/robot/backup/snake_with_dummy.xacro (robot description, xacro)
@@ -109,24 +109,24 @@
     </xacro:macro>
 	<!-- * * * Link Definitions * * * -->
-<link name="startpt">
- 	<inertial>
-            <origin xyz="1 0 0.075" rpy="0 0 0"/>
-            <mass value="0.1" />
-            <inertia ixx="0.00025" ixy="0.0" ixz="0.0" iyy="0.00025" iyz="0.0" izz="0.000125"/>
+    <link name="startpt">
+	<inertial>
+            <origin xyz="0 0 0.075" rpy="0 0 0"/>
+            <mass value="0.01" />
+            <inertia ixx="0.00001" ixy="0.0" ixz="0.0" iyy="0.00001" iyz="0.0" izz="0.00001"/>
         </inertial>
         <collision>
             <origin xyz="1 0 0.075" rpy="0 0 0"/>
             <geometry>
-                <cylinder radius="0.008" length="0.5"/>
+                <cylinder radius="0.08" length="0.5"/>
             </geometry>
         </collision>
         <visual>
-            <origin xyz="1 0 0.075" rpy="0 0 0"/>
+            <origin xyz="5 5 0.2" rpy="0 0 0"/>
             <geometry>
-                <cylinder radius="0.008" length="0.5"/>
+                <cylinder radius="0.008" length="0.01"/>
             </geometry>
         </visual>
 	</link>
-<gazebo reference="startpt">
+    <gazebo reference="startpt">
         <kp>100000000000000.0</kp>
         <kd>100000000000000.0</kd>
@@ -163,7 +163,7 @@
         <self_collide>1</self_collide>
     </gazebo>
-<joint name="noreal" type="floating">
+    <joint name="noreal" type="floating">
     	    <parent link="startpt"/>
-        	<child link="base_link"/>
+            <child link="base_link"/>
             <origin xyz="0 0 0" rpy="0 0 0"/>
     </joint>

Commit message: dummylink

File: snake_description2/robot/backup/snake_with_dummy.xacro (robot description, xacro)
@@ -111,18 +111,18 @@
     <link name="startpt">
 	<inertial>
-            <origin xyz="0 0 0.075" rpy="0 0 0"/>
+            <origin xyz="0 0 0.005" rpy="0 0 0"/>
             <mass value="0.01" />
             <inertia ixx="0.00001" ixy="0.0" ixz="0.0" iyy="0.00001" iyz="0.0" izz="0.00001"/>
         </inertial>
         <collision>
-            <origin xyz="1 0 0.075" rpy="0 0 0"/>
+            <origin xyz="0 0 0.005" rpy="0 0 0"/>
             <geometry>
-                <cylinder radius="0.08" length="0.5"/>
+                <cylinder radius="0.05" length="0.1"/>
             </geometry>
         </collision>
         <visual>
-            <origin xyz="5 5 0.2" rpy="0 0 0"/>
+            <origin xyz="0 0 0.005" rpy="0 0 0"/>
             <geometry>
-                <cylinder radius="0.008" length="0.01"/>
+                <cylinder radius="0.05" length="0.01"/>
             </geometry>
         </visual>
@@ -143,13 +143,13 @@
         </inertial>
         <collision>
-            <origin xyz="0 0 0.075" rpy="0 0 0"/>
+            <origin xyz="0 0 0.08" rpy="0 0 0"/>
             <geometry>
-                <cylinder radius="0.05" length="0.15"/>
+                <cylinder radius="0.05" length="0.14"/>
             </geometry>
         </collision>
         <visual>
-            <origin xyz="0 0 0.075" rpy="0 0 0"/>
+            <origin xyz="0 0 0.08" rpy="0 0 0"/>
             <geometry>
-                <cylinder radius="0.05" length="0.15"/>
+                <cylinder radius="0.05" length="0.14"/>
             </geometry>
         </visual>
@@ -163,8 +163,8 @@
         <self_collide>1</self_collide>
     </gazebo>
-    <joint name="noreal" type="floating">
+    <joint name="noreal" type="fixed">
     	    <parent link="startpt"/>
             <child link="base_link"/>
-            <origin xyz="0 0 0" rpy="0 0 0"/>
+            <origin xyz="0 0 0.01" rpy="0 0 0"/>
     </joint>
     <xacro:body_link base_name="snake_body_1" parent_name="base_link" colour="Blue" xx="1"  yy="0" />

File: snake_description2/robot/snake_controllers.urdf.xacro (robot description, xacro)
@@ -6,4 +6,14 @@
         </plugin>
     </gazebo>
+<plugin name="p3d_base_controller" filename="libgazebo_ros_p3d.so">
+  <alwaysOn>true</alwaysOn>
+  <updateRate>5.0</updateRate>
+  <bodyName>base_link</bodyName>
+  <topicName>odom</topicName>
+  <gaussianNoise>0.01</gaussianNoise>
+  <frameName>startpt</frameName>
+  <xyzOffsets>0 0 0</xyzOffsets>
+  <rpyOffsets>0 0 0</rpyOffsets>
+</plugin>
     <!-- MACROS -->
     <xacro:macro name="body_link" params="base_name parent_name colour xx yy">
@@ -99,4 +109,31 @@
     </xacro:macro>
 	<!-- * * * Link Definitions * * * -->
+    <link name="startpt">
+	<inertial>
+            <origin xyz="0 0 0.005" rpy="0 0 0"/>
+            <mass value="0.01" />
+            <inertia ixx="0.00001" ixy="0.0" ixz="0.0" iyy="0.00001" iyz="0.0" izz="0.00001"/>
+        </inertial>
+        <collision>
+            <origin xyz="0 0 0.001" rpy="0 0 0"/>
+            <geometry>
+                <cylinder radius="0.05" length="0.002"/>
+            </geometry>
+        </collision>
+        <visual>
+            <origin xyz="0 0 0.001" rpy="0 0 0"/>
+            <geometry>
+                <cylinder radius="0.05" length="0.002"/>
+            </geometry>
+        </visual>
+	</link>
+    <gazebo reference="startpt">
+        <kp>100000000000000.0</kp>
+        <kd>100000000000000.0</kd>
+        <mu1>10.0</mu1>
+        <mu2>10.0</mu2>
+        <material>Gazebo/Black</material>
+        <self_collide>0</self_collide>
+    </gazebo>
     <link name="base_link">
  	    <inertial>
@@ -126,4 +163,9 @@
         <self_collide>1</self_collide>
     </gazebo>
+    <joint name="noreal" type="fixed">
+    	    <parent link="startpt"/>
+            <child link="base_link"/>
+            <origin xyz="0 0 0.002" rpy="0 0 0"/>
+    </joint>
     <xacro:body_link base_name="snake_body_1" parent_name="base_link" colour="Blue" xx="1"  yy="0" />
     <xacro:body_link base_name="snake_body_2" parent_name="snake_body_1" colour="Red" xx="1" yy="0" />
