Commit message: prove

File: snake_description2/robot/snake_controllers_n.urdfcav.xacro (robot description, xacro)
@@ -6,16 +6,16 @@
         </plugin>
     </gazebo>
-<plugin name="p3d_base_controller" filename="libgazebo_ros_p3d.so">
-  <alwaysOn>true</alwaysOn>
-  <updateRate>5.0</updateRate>
-  <bodyName>base_link</bodyName>
-  <topicName>odom</topicName>
-  <gaussianNoise>0.01</gaussianNoise>
-  <frameName>startpt</frameName>
-  <xyzOffsets>0 0 0</xyzOffsets>
-  <rpyOffsets>0 0 0</rpyOffsets>
-</plugin>
     <!-- MACROS -->
-    <xacro:macro name="body_link" params="base_name parent_name colour xx yy">
+    <xacro:property name="NumberOfElements" value="$(arg prefix)" />
+    <xacro:macro name="loop" params="links_qty">
+        <xacro:if value="${links_qty == 3}">
+            <xacro:body_link base_name="snake_body_${links_qty-1}" parent_name="snake_body_${links_qty}" colour="Red"/>
+            <xacro:if value="${links_qty}">
+                <xacro:loop links_qty="${links_qty-1}" />
+            </xacro:if>
+        </xacro:if>
+    </xacro:macro>
+    <xacro:loop links_qty="${NumberOfElements}" />
+    <xacro:macro name="body_link" params="base_name parent_name colour">
         <link name="${base_name}_aux">
             <inertial>
@@ -43,5 +43,5 @@
             <mu2>10.0</mu2>
             <material>Gazebo/Black</material>
-            <self_collide>0</self_collide>
+            <self_collide>1</self_collide>
         </gazebo>
         <link name="${base_name}">
@@ -85,5 +85,5 @@
             <origin xyz="0 0 0.05" rpy="0 0 0"/>
             <limit lower="-1.8008" upper="1.8008" effort="20.0" velocity="3"/>
-            <axis xyz="${xx} ${yy} 0"/>
+            <axis xyz="1 0 0"/>
     	</joint>
 	    <transmission name="tran${base_name}_aux">
@@ -109,51 +109,24 @@
     </xacro:macro>
 	<!-- * * * Link Definitions * * * -->
-    <link name="startpt">
-	<inertial>
-            <origin xyz="0 0 0.005" rpy="0 0 0"/>
-            <mass value="0.01" />
-            <inertia ixx="0.00001" ixy="0.0" ixz="0.0" iyy="0.00001" iyz="0.0" izz="0.00001"/>
-        </inertial>
-        <collision>
-            <origin xyz="0 0 0.001" rpy="0 0 0"/>
-            <geometry>
-                <cylinder radius="0.05" length="0.002"/>
-            </geometry>
-        </collision>
-        <visual>
-            <origin xyz="0 0 0.001" rpy="0 0 0"/>
-            <geometry>
-                <cylinder radius="0.05" length="0.002"/>
-            </geometry>
-        </visual>
+	<link name="snake_body_${NumberOfElements}">
+     	    <inertial>
+                <origin xyz="0 0 0.075" rpy="0 0 0"/>
+                <mass value="0.1" />
+                <inertia ixx="0.00025" ixy="0.0" ixz="0.0" iyy="0.00025" iyz="0.0" izz="0.000125"/>
+            </inertial>
+            <collision>
+                <origin xyz="0 0 0.075" rpy="0 0 0"/>
+                <geometry>
+                    <cylinder radius="0.05" length="0.15"/>
+                </geometry>
+            </collision>
+            <visual>
+                <origin xyz="0 0 0.075" rpy="0 0 0"/>
+                <geometry>
+                    <cylinder radius="0.05" length="0.15"/>
+                </geometry>
+            </visual>
 	</link>
-    <gazebo reference="startpt">
-        <kp>100000000000000.0</kp>
-        <kd>100000000000000.0</kd>
-        <mu1>10.0</mu1>
-        <mu2>10.0</mu2>
-        <material>Gazebo/Black</material>
-        <self_collide>1</self_collide>
-    </gazebo>
-    <link name="base_link">
- 	    <inertial>
-            <origin xyz="0 0 0.075" rpy="0 0 0"/>
-            <mass value="0.1" />
-            <inertia ixx="0.00025" ixy="0.0" ixz="0.0" iyy="0.00025" iyz="0.0" izz="0.000125"/>
-        </inertial>
-        <collision>
-            <origin xyz="0 0 0.075" rpy="0 0 0"/>
-            <geometry>
-                <cylinder radius="0.05" length="0.15"/>
-            </geometry>
-        </collision>
-        <visual>
-            <origin xyz="0 0 0.075" rpy="0 0 0"/>
-            <geometry>
-                <cylinder radius="0.05" length="0.15"/>
-            </geometry>
-        </visual>
-	</link>
-    <gazebo reference="base_link">
+    <gazebo reference="snake_body_${NumberOfElements}">
         <kp>100000000000000.0</kp>
         <kd>100000000000000.0</kd>
@@ -163,15 +136,12 @@
         <self_collide>1</self_collide>
     </gazebo>
-    <joint name="noreal" type="fixed">
-    	    <parent link="startpt"/>
-            <child link="base_link"/>
-            <origin xyz="0 0 0.002" rpy="0 0 0"/>
-    </joint>
-    <xacro:body_link base_name="snake_body_1" parent_name="base_link" colour="Blue" xx="1"  yy="0" />
-    <xacro:body_link base_name="snake_body_2" parent_name="snake_body_1" colour="Red" xx="1" yy="0" />
-    <xacro:body_link base_name="snake_body_3" parent_name="snake_body_2" colour="Purple" xx="1" yy="0" />
-    <xacro:body_link base_name="snake_body_4" parent_name="snake_body_3" colour="White" xx="1" yy="0" />
-    <xacro:body_link base_name="snake_body_5" parent_name="snake_body_4" colour="Yellow" xx="1" yy="0"  />
-    <xacro:body_link base_name="snake_body_6" parent_name="snake_body_5" colour="Turquoise" xx="1" yy="0" />
-    <xacro:body_link base_name="snake_body_7" parent_name="snake_body_6" colour="Grey" xx="1" yy="0" />
+    <!--
+    <xacro:body_link base_name="snake_body_1" parent_name="snake_body_0" colour="Blue"/>
+    <xacro:body_link base_name="snake_body_2" parent_name="snake_body_1" colour="Red"/>
+    <xacro:body_link base_name="snake_body_3" parent_name="snake_body_2" colour="Purple"/>
+    <xacro:body_link base_name="snake_body_4" parent_name="snake_body_3" colour="White"/>
+    <xacro:body_link base_name="snake_body_5" parent_name="snake_body_4" colour="Yellow"/>
+    <xacro:body_link base_name="snake_body_6" parent_name="snake_body_5" colour="Turquoise"/>
+    <xacro:body_link base_name="snake_body_7" parent_name="snake_body_6" colour="Grey"/>
+    -->
 </robot>
