Commit message: parametric

File: snake_description/robot/snake_controllers_n.urdf.xacro (robot description, xacro)
@@ -7,15 +7,24 @@
     </gazebo>
     <!-- MACROS -->
+    <xacro:property name="NumberOfElements" value="$(arg prefix)" />
+    <xacro:property name="Radius" value="$(arg diam)" />
+    <xacro:property name="Lenght_tot" value="$(arg leng)" />
+    <xacro:property name="Lenght" value="${Lenght_tot-0.05}" />
+    <xacro:property name="Mass_tot" value="$(arg mass)" />
+    <xacro:property name="Mass1" value="${Mass_tot*Lenght/Lenght_tot}" />
+    <xacro:property name="Mass2" value="${Mass_tot*0.05/Lenght_tot}" />
+    <xacro:property name="mu" value="$(arg friction)" />
+    <xacro:property name="maxeffort" value="$(arg max_effort)" />
     <xacro:macro name="body_link" params="base_name parent_name colour">
         <link name="${base_name}_aux">
             <inertial>
                 <origin xyz="0 0 0.025" rpy="0 0 0"/>
-                <mass value="0.1" />
-                <inertia ixx="0.00025" ixy="0.0" ixz="0.0" iyy="0.00025" iyz="0.0" izz="0.000125"/>
+                <mass value="${Mass2}" />
+                <inertia ixx="${(Radius*Radius/4+0.05*0.05/12)*Mass2}" ixy="0.0" ixz="0.0" iyy="${(Radius*Radius/4+0.05*0.05/12)*Mass2}" iyz="0.0" izz="${Mass2*Radius*Radius/2}"/>
             </inertial>
             <collision>
                 <origin xyz="0 0 0.025" rpy="0 0 0"/>
                 <geometry>
-                    <cylinder radius="0.05" length="0.05"/>
+                    <cylinder radius="${Radius}" length="0.05"/>
                 </geometry>
             </collision>
@@ -23,5 +32,5 @@
                 <origin xyz="0 0 0.025" rpy="0 0 0"/>
                 <geometry>
-                    <cylinder radius="0.05" length="0.05"/>
+                    <cylinder radius="${Radius}" length="0.05"/>
                 </geometry>
             </visual>
@@ -30,25 +39,25 @@
             <kp>1000000000.0</kp>
             <kd>1000000000.0</kd>
-            <mu1>10.0</mu1>
-            <mu2>10.0</mu2>
+            <mu1>${mu}</mu1>
+            <mu2>${mu}</mu2>
             <material>Gazebo/Black</material>
-            <self_collide>1</self_collide>
+            <self_collide>0</self_collide>
         </gazebo>
         <link name="${base_name}">
      	    <inertial>
-                <origin xyz="0 0 0.075" rpy="0 0 0"/>
-                <mass value="0.1" />
-                <inertia ixx="0.00025" ixy="0.0" ixz="0.0" iyy="0.00025" iyz="0.0" izz="0.000125"/>
+                <origin xyz="0 0 ${Lenght/2}" rpy="0 0 0"/>
+                <mass value="${Mass1}" />
+                <inertia ixx="${(Radius*Radius/4+Lenght*Lenght/12)*Mass1}" ixy="0.0" ixz="0.0" iyy="${(Radius*Radius/4+Lenght*Lenght/12)*Mass1}" iyz="0.0" izz="${Mass1*Radius*Radius/2}"/>
             </inertial>
             <collision>
-                <origin xyz="0 0 0.075" rpy="0 0 0"/>
+                <origin xyz="0 0 ${Lenght/2}" rpy="0 0 0"/>
                 <geometry>
-                    <cylinder radius="0.05" length="0.15"/>
+                    <cylinder radius="${Radius}" length="${Lenght}"/>
                 </geometry>
             </collision>
             <visual>
-                <origin xyz="0 0 0.075" rpy="0 0 0"/>
+                <origin xyz="0 0 ${Lenght/2}" rpy="0 0 0"/>
                 <geometry>
-                    <cylinder radius="0.05" length="0.15"/>
+                    <cylinder radius="${Radius}" length="${Lenght}"/>
                 </geometry>
             </visual>
@@ -57,8 +66,8 @@
             <kp>1000000000.0</kp>
             <kd>1000000000.0</kd>
-            <mu1>10.0</mu1>
-            <mu2>10.0</mu2>
+            <mu1>${mu}</mu1>
+            <mu2>${mu}</mu2>
             <material>Gazebo/${colour}</material>
-            <self_collide>1</self_collide>
+            <self_collide>0</self_collide>
         </gazebo>
         <!-- We add to the Origin displacement a margin for flex due to self colisions for parent_name and base_name-->
@@ -66,7 +75,7 @@
             <parent link="${parent_name}"/>
         	<child link="${base_name}_aux"/>
-            <origin xyz="0 0 0.15" rpy="0 0 0"/>
-            <limit lower="-1.5708" upper="1.5708" effort="100.0" velocity="0.5"/>
-            <axis xyz="1 0 0"/>
+            <origin xyz="0 0 ${Lenght}" rpy="0 0 0"/>
+            <limit lower="-1.5708" upper="1.5708" effort="${maxeffort}" velocity="0.5"/>
+            <axis xyz="0 0 1"/>
     	</joint>
         <joint name="${base_name}_joint" type="revolute">
@@ -74,6 +83,6 @@
         	<child link="${base_name}"/>
             <origin xyz="0 0 0.05" rpy="0 0 0"/>
-            <limit lower="-1.5708" upper="1.5708" effort="100.0" velocity="0.5"/>
-            <axis xyz="0 1 0"/>
+            <limit lower="-1.5708" upper="1.5708" effort="${maxeffort}" velocity="0.5"/>
+            <axis xyz="1 0 0"/>
     	</joint>
 	    <transmission name="tran${base_name}_aux">
@@ -98,5 +107,4 @@
         </transmission>
     </xacro:macro>
-    <xacro:property name="NumberOfElements" value="$(arg prefix)" />
     <xacro:macro name="loop" params="links_qty">
         <xacro:if value="${links_qty > 0}">
@@ -111,5 +119,5 @@
 	<inertial>
             <origin xyz="0 0 0.005" rpy="0 0 0"/>
-            <mass value="0.01" />
+            <mass value="0.0001" />
             <inertia ixx="0.00001" ixy="0.0" ixz="0.0" iyy="0.00001" iyz="0.0" izz="0.00001"/>
         </inertial>
@@ -117,5 +125,5 @@
             <origin xyz="0 0 0.001" rpy="0 0 0"/>
             <geometry>
-                <cylinder radius="0.05" length="0.002"/>
+                <cylinder radius="${Radius}" length="0.002"/>
             </geometry>
         </collision>
@@ -123,5 +131,5 @@
             <origin xyz="0 0 0.001" rpy="0 0 0"/>
             <geometry>
-                <cylinder radius="0.05" length="0.002"/>
+                <cylinder radius="${Radius}" length="0.002"/>
             </geometry>
         </visual>
@@ -130,8 +138,8 @@
         <kp>100000000000000.0</kp>
         <kd>100000000000000.0</kd>
-        <mu1>10.0</mu1>
-        <mu2>10.0</mu2>
+        <mu1>${mu}</mu1>
+        <mu2>${mu}</mu2>
         <material>Gazebo/Black</material>
-        <self_collide>1</self_collide>
+        <self_collide>0</self_collide>
     </gazebo>
  <joint name="noreal" type="fixed">
@@ -141,19 +149,19 @@
     </joint>
 	<link name="snake_body_${NumberOfElements}">
-     	    <inertial>
-                <origin xyz="0 0 0.075" rpy="0 0 0"/>
-                <mass value="0.1" />
-                <inertia ixx="0.00025" ixy="0.0" ixz="0.0" iyy="0.00025" iyz="0.0" izz="0.000125"/>
+     	   <inertial>
+                <origin xyz="0 0 ${Lenght/2}" rpy="0 0 0"/>
+                <mass value="${Mass1}" />
+                <inertia ixx="${(Radius*Radius/4+Lenght*Lenght/12)*Mass1}" ixy="0.0" ixz="0.0" iyy="${(Radius*Radius/4+Lenght*Lenght/12)*Mass1}" iyz="0.0" izz="${Mass1*Radius*Radius/2}"/>
             </inertial>
             <collision>
-                <origin xyz="0 0 0.075" rpy="0 0 0"/>
+                <origin xyz="0 0 ${Lenght/2}" rpy="0 0 0"/>
                 <geometry>
-                    <cylinder radius="0.05" length="0.15"/>
+                    <cylinder radius="${Radius}" length="${Lenght}"/>
                 </geometry>
             </collision>
             <visual>
-                <origin xyz="0 0 0.075" rpy="0 0 0"/>
+                <origin xyz="0 0 ${Lenght/2}" rpy="0 0 0"/>
                 <geometry>
-                    <cylinder radius="0.05" length="0.15"/>
+                    <cylinder radius="${Radius}" length="${Lenght}"/>
                 </geometry>
             </visual>
@@ -162,8 +170,8 @@
         <kp>100000000000000.0</kp>
         <kd>100000000000000.0</kd>
-        <mu1>10.0</mu1>
-        <mu2>10.0</mu2>
+        <mu1>${mu}</mu1>
+        <mu2>${mu}</mu2>
         <material>Gazebo/White</material>
-        <self_collide>1</self_collide>
+        <self_collide>0</self_collide>
     </gazebo>
     <xacro:loop links_qty="${NumberOfElements}" />

Commit message: new

File: snake_description/robot/snake_controllers_n.urdf.xacro (robot description, xacro)
@@ -16,4 +16,5 @@
     <xacro:property name="mu" value="$(arg friction)" />
     <xacro:property name="maxeffort" value="$(arg max_effort)" />
+    <xacro:property name="max_ef_yaw" value="$(arg max_yaw)" />
     <xacro:macro name="body_link" params="base_name parent_name colour">
         <link name="${base_name}_aux">
@@ -76,5 +77,5 @@
         	<child link="${base_name}_aux"/>
             <origin xyz="0 0 ${Lenght}" rpy="0 0 0"/>
-            <limit lower="-1.5708" upper="1.5708" effort="${maxeffort}" velocity="0.5"/>
+            <limit lower="-1.5708" upper="1.5708" effort="${max_ef_yaw}" velocity="0.5"/>
             <axis xyz="0 0 1"/>
     	</joint>
@@ -147,5 +148,5 @@
             <child link="snake_body_${NumberOfElements}"/>
             <origin xyz="0 0 0.002" rpy="0 0 0"/>
-            <limit lower="-100" upper="100" effort="${maxeffort}" velocity="0.5"/>
+            <limit lower="-100" upper="100" effort="0.1" velocity="0.5"/>
             <axis xyz="0 0 1"/>
     </joint>

Commit message: semi_def

File: snake_description/robot/snake_controllers_n.urdf.xacro (robot description, xacro)
@@ -27,5 +27,5 @@
                 <origin xyz="0 0 0.025" rpy="0 0 0"/>
                 <geometry>
-                    <cylinder radius="${Radius}" length="0.05"/>
+                    <cylinder radius="${Radius-0.005}" length="0.05"/>
                 </geometry>
             </collision>
@@ -33,5 +33,5 @@
                 <origin xyz="0 0 0.025" rpy="0 0 0"/>
                 <geometry>
-                    <cylinder radius="${Radius}" length="0.05"/>
+                    <cylinder radius="${Radius-0.005}" length="0.05"/>
                 </geometry>
             </visual>
